File: KiCAD files/DremelLevelSensor.kicad_pcb (KiCad board)
At the start: 2 copper layers, 11 x 22 mm, 6 parts

Commit message: Update PCB and Schematic to remove unnecessary jumper that was added to try to get DKRed to work
Parts:
- removed JP3: SolderJumper_2_Open, Jumper:SolderJumper-2_P1.3mm_Open_RoundedPad1.0x1.5mm
Other:
- board text removed: "WayWayWay"
